Commit message: Finished Hw 2

File: ros_ws/src/homework/Hw2/fourWheelRobot/urdf/lidar.xacro (robot description, xacro)
@@ -36,5 +36,6 @@
             <update_rate>10</update_rate>
             <always_on>true</always_on>
-            <visualize>true</visualize>
+            <!-- Drawing the rays is expensive without a GPU; see the scan in RViz instead -->
+            <visualize>false</visualize>
             <lidar>
                 <scan>

File: ros_ws/src/homework/Hw2/fourWheelRobot/urdf/my_robot.urdf (robot description, URDF)
Before this commit: robot my_robot, 5 links, 4 joints
Links:
- added link lidar_link, mass 1.5; collision cylinder length=0.3 radius=0.1875; visual cylinder length=0.3 radius=0.1875
- link back_left_wheel: mass 0.2 -> 0.025; geometry collision cylinder length=0.03 radius=0.04
- link back_right_wheel: mass 0.2 -> 0.025; geometry collision cylinder length=0.03 radius=0.04
- link base_link: mass 2.0 -> 9.0; geometry collision box size=2.25 1.5 0.45; visual box size=0.15 0.15 1.125
- link front_left_wheel: mass 0.2 -> 0.025; geometry collision cylinder length=0.03 radius=0.04
- link front_right_wheel: mass 0.2 -> 0.025; geometry collision cylinder length=0.03 radius=0.04
Joints:
- added joint lidar_joint: type fixed, parent base_link, child lidar_link, origin xyz=0.6 0 0.8625 rpy=0 0 0
- joint back_left_wheel_joint: origin xyz=-0.1 0.115 0 rpy=-1.5708 0 0 -> xyz=-1.05 0.6375 -0.5625 rpy=-1.5708 0 0
- joint back_right_wheel_joint: origin xyz=-0.1 -0.115 0 rpy=-1.5708 0 0 -> xyz=-1.05 -0.6375 -0.5625 rpy=-1.5708 0 0
- joint front_left_wheel_joint: origin xyz=0.1 0.115 0 rpy=-1.5708 0 0 -> xyz=1.05 0.6375 -0.5625 rpy=-1.5708 0 0
- joint front_right_wheel_joint: origin xyz=0.1 -0.115 0 rpy=-1.5708 0 0 -> xyz=1.05 -0.6375 -0.5625 rpy=-1.5708 0 0
